File: electronics/elite dangerous keypad.kicad_pcb (KiCad board)
At the start: 2 copper layers, 3 parts, among them U1 MCP23018x-x-SP, U2 MCP23018x-x-SP

Commit message: schematic for cardboard box version
Parts:
- removed U2: MCP23018x-x-SP, Package_DIP:DIP-28_W7.62mm
- added J1: button, Connector_PinHeader_2.54mm:PinHeader_1x16_P2.54mm_Vertical, F.Cu at (177.2, 40.0)
- added J3: swd debug, Connector_PinHeader_2.54mm:PinHeader_1x04_P2.54mm_Vertical, F.Cu at (258.5, 69.2)
- added J4: led, Connector_PinHeader_2.54mm:PinHeader_1x16_P2.54mm_Vertical, F.Cu at (179.7, 101.0)
- added J6: Conn_01x02, Connector_PinSocket_2.54mm:PinSocket_1x02_P2.54mm_Vertical, F.Cu at (230.0, 40.0)
- added R11: R, Resistor_THT:R_Axial_DIN0204_L3.6mm_D1.6mm_P7.62mm_Horizontal, F.Cu at (179.7, 89.6)
- added R12: R, Resistor_THT:R_Axial_DIN0204_L3.6mm_D1.6mm_P7.62mm_Horizontal, F.Cu at (182.3, 89.6)
- added R13: R, Resistor_THT:R_Axial_DIN0204_L3.6mm_D1.6mm_P7.62mm_Horizontal, F.Cu at (184.8, 89.6)
- added R14: R, Resistor_THT:R_Axial_DIN0204_L3.6mm_D1.6mm_P7.62mm_Horizontal, F.Cu at (187.4, 89.6)
- added R15: R, Resistor_THT:R_Axial_DIN0204_L3.6mm_D1.6mm_P7.62mm_Horizontal, F.Cu at (189.9, 89.6)
- added R16: R, Resistor_THT:R_Axial_DIN0204_L3.6mm_D1.6mm_P7.62mm_Horizontal, F.Cu at (192.4, 89.6)
- added R17: R, Resistor_THT:R_Axial_DIN0204_L3.6mm_D1.6mm_P7.62mm_Horizontal, F.Cu at (195.0, 89.6)
- added R18: R, Resistor_THT:R_Axial_DIN0204_L3.6mm_D1.6mm_P7.62mm_Horizontal, F.Cu at (197.5, 89.6)
- added R19: R, Resistor_THT:R_Axial_DIN0204_L3.6mm_D1.6mm_P7.62mm_Horizontal, F.Cu at (200.1, 89.6)
- added R20: R, Resistor_THT:R_Axial_DIN0204_L3.6mm_D1.6mm_P7.62mm_Horizontal, F.Cu at (202.6, 89.6)
- added R21: R, Resistor_THT:R_Axial_DIN0204_L3.6mm_D1.6mm_P7.62mm_Horizontal, F.Cu at (205.1, 89.6)
- added R22: R, Resistor_THT:R_Axial_DIN0204_L3.6mm_D1.6mm_P7.62mm_Horizontal, F.Cu at (207.7, 89.6)
- added R23: R, Resistor_THT:R_Axial_DIN0204_L3.6mm_D1.6mm_P7.62mm_Horizontal, F.Cu at (210.2, 89.6)
- added R24: R, Resistor_THT:R_Axial_DIN0204_L3.6mm_D1.6mm_P7.62mm_Horizontal, F.Cu at (212.8, 89.6)
- added R25: R, Resistor_THT:R_Axial_DIN0204_L3.6mm_D1.6mm_P7.62mm_Horizontal, F.Cu at (215.3, 89.6)
- added R26: R, Resistor_THT:R_Axial_DIN0204_L3.6mm_D1.6mm_P7.62mm_Horizontal, F.Cu at (217.8, 89.6)
- added R5: 1k5, Resistor_THT:R_Axial_DIN0204_L3.6mm_D1.6mm_P2.54mm_Vertical, F.Cu at (195.0, 59.2)
- added R6: 1k5, Resistor_THT:R_Axial_DIN0204_L3.6mm_D1.6mm_P2.54mm_Vertical, F.Cu at (198.1, 59.2)
- added U3: MCP23018x-x-SP, Package_DIP:DIP-28_W7.62mm, F.Cu at (217.8, 83.2)
- A1: value Arduino_Pro_Micro -> Tiny2040
- moved A1 107.4 mm to (245.5, 37.2)
- moved U1 74.7 mm to (192.4, 84.5), turned to 180 degrees
Connections:
- A1 pad 1: unconnected-(A1-D1/TX-Pad1) -> +5V
- A1 pad 10: /INPUT_INTB -> /MCU_INPUT_INT
- A1 pad 11: unconnected-(A1-D8/A8-Pad11) -> /SCL
- A1 pad 12: unconnected-(A1-D9/A9-Pad12) -> /SDA
- A1 pad 16: +5V -> unconnected-(A1-0-Pad16)
- A1 pad 2: unconnected-(A1-D0/RX-Pad2) -> GND
- A1 pad 5: /SDA -> unconnected-(A1-A2/28-Pad5)
- A1 pad 6: /SCL -> unconnected-(A1-A1/27-Pad6)
- A1 pad 8: /INPUT_INTA -> unconnected-(A1-GND-Pad8)
- U1 pad 10: unconnected-(U1-GPB7-Pad10) -> /B15
- U1 pad 16: unconnected-(U1-~{RESET}-Pad16) -> +5V
- U1 pad 18: /INPUT_INTB -> unconnected-(U1-INTB-Pad18)
- U1 pad 19: /INPUT_INTA -> /MCU_INPUT_INT
- U1 pad 20: Net-(SW1-A) -> /B0
- U1 pad 21: unconnected-(U1-GPA1-Pad21) -> /B1
- U1 pad 22: unconnected-(U1-GPA2-Pad22) -> /B2
- U1 pad 23: unconnected-(U1-GPA3-Pad23) -> /B3
- U1 pad 24: unconnected-(U1-GPA4-Pad24) -> /B4
- U1 pad 25: unconnected-(U1-GPA5-Pad25) -> /B5
- U1 pad 26: unconnected-(U1-GPA6-Pad26) -> /B6
- U1 pad 27: unconnected-(U1-GPA7-Pad27) -> /B7
- U1 pad 3: unconnected-(U1-GPB0-Pad3) -> /B8
- U1 pad 4: unconnected-(U1-GPB1-Pad4) -> /B9
- U1 pad 5: unconnected-(U1-GPB2-Pad5) -> /B10
- U1 pad 6: unconnected-(U1-GPB3-Pad6) -> /B11
- U1 pad 7: unconnected-(U1-GPB4-Pad7) -> /B12
- U1 pad 8: unconnected-(U1-GPB5-Pad8) -> /B13
- U1 pad 9: unconnected-(U1-GPB6-Pad9) -> /B14
Routing:
- net /L0: track 0.00 -> 46.7 mm
- net /L15: track 0.00 -> 46.6 mm
- net /B7: track 0.00 -> 46.1 mm
- net /L14: track 0.00 -> 44.9 mm
- net /B8: track 0.00 -> 44.1 mm
- net /B6: track 0.00 -> 43.1 mm
- net /B9: track 0.00 -> 42.8 mm
- net /B10: track 0.00 -> 41.2 mm
- net /L13: track 0.00 -> 40.9 mm
- net /B11: track 0.00 -> 40.3 mm
- net /B5: track 0.00 -> 38.9 mm
- net /L12: track 0.00 -> 37.2 mm
- net /B12: track 0.00 -> 35.5 mm, vias 0 -> 1
- net /B4: track 0.00 -> 35.3 mm
- net /B13: track 0.00 -> 34.1 mm, vias 0 -> 1
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